File: PCB/Car/Car.kicad_pcb (KiCad board)
At the start: 2 copper layers, 70 x 100 mm, 10 parts, among them J1 L1, J2 L2, J3 R1, J4 R2, J5 Conn_01x02_Pin, J6 Conn_01x02_Pin, J7 Conn_01x03, J8 Conn_01x06, U2 YAAJ_DCDC_StepDown_LM2596, U3 YAAJ_DCDC_StepDown_LM2596

Commit message: finish PCB
Parts:
- removed U2: YAAJ_DCDC_StepDown_LM2596, lm2596:YAAJ_DCDC_StepDown_LM2596
- added J10: FL2, Connector:JWT_A3963_1x02_P3.96mm_Vertical, F.Cu at (30.9, 182.6)
- added J10: Conn_01x12, Connector_PinHeader_2.54mm:PinHeader_1x12_P2.54mm_Vertical, F.Cu at (18.8, 134.3)
- added J11: Conn_01x03, Connector:FanPinHeader_1x03_P2.54mm_Vertical, F.Cu at (24.7, 142.8)
- added J11: FLT, Connector:JWT_A3963_1x02_P3.96mm_Vertical, F.Cu at (30.9, 192.3)
- added J12: Conn_01x03, Connector:FanPinHeader_1x03_P2.54mm_Vertical, F.Cu at (24.7, 134.8)
- added J9: Conn_01x06, Connector_PinHeader_2.54mm:PinHeader_1x06_P2.54mm_Vertical, F.Cu at (16.8, 190.3)
- added J9: FL1, Connector:JWT_A3963_1x02_P3.96mm_Vertical, F.Cu at (30.9, 173.3)
- J1, J2, J3, J4: footprint Connector_JST:JST_PH_S2B-PH-K_1x02_P2.00mm_Horizontal -> Connector:JWT_A3963_1x02_P3.96mm_Vertical
- J5: value Conn_01x02_Pin -> R1+2; footprint Connector_JST:JST_PH_S2B-PH-K_1x02_P2.00mm_Horizontal -> Connector:JWT_A3963_1x02_P3.96mm_Vertical
- J6: value Conn_01x02_Pin -> L1+2; footprint Connector_JST:JST_PH_S2B-PH-K_1x02_P2.00mm_Horizontal -> Connector:JWT_A3963_1x02_P3.96mm_Vertical
- J7: footprint Connector_JST:JST_PH_B3B-PH-K_1x03_P2.00mm_Vertical -> Connector:FanPinHeader_1x03_P2.54mm_Vertical
- J8: value Conn_01x06 -> Conn_01x04; footprint Connector_JST:JST_PH_B6B-PH-K_1x06_P2.00mm_Vertical -> Connector:FanPinHeader_1x04_P2.54mm_Vertical
- moved J8 154.2 mm to (27.3, 149.7), turned to -90 degrees
- moved J2 127.9 mm to (49.9, 182.9)
- moved J6 126.1 mm to (49.9, 192.3)
- moved J4 122.0 mm to (40.4, 182.6)
- moved J5 120.1 mm to (40.4, 192.3)
- moved J1 116.6 mm to (49.9, 173.3)
- moved J3 111.1 mm to (40.4, 173.3)
- moved J7 110.9 mm to (24.7, 126.8)
- moved U3 74.6 mm to (36.4, 166.1)
Connections:
- net +6V renamed +6.5V
- J8 pad 1: GND -> IN4
- J8 pad 2: +5V -> IN3
- J8 pad 3: IN4 -> IN2
- J8 pad 4: IN3 -> IN1
Routing:
- net BA: track 0.00 -> 55.5 mm
- net +5V: track 131.1 -> 77.7 mm
- net VCC: track 52.5 -> 0.00 mm
- net BB: track 0.00 -> 50.6 mm
- net AA: track 0.00 -> 38.9 mm
- net +6.5V: track 57.4 -> 91.8 mm
- net AB: track 0.00 -> 34.0 mm
- net Net-(J10-Pin_2): track 0.00 -> 19.3 mm
- net Net-(J10-Pin_1): track 0.00 -> 19.3 mm
- net GND: track 245.2 -> 232.4 mm
- net Net-(J3-Pin_2): track 30.9 -> 19.0 mm
- net Net-(J1-Pin_2): track 30.8 -> 19.0 mm
- net LED1: track 0.00 -> 11.0 mm
- net LED2: track 0.00 -> 9.91 mm
- net IN2: track 0.00 -> 8.56 mm
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- added copper zone on B.Cu, net GND
- added copper zone on F.Cu, net GND
Other:
- board size 70 x 100 mm -> 45.5 x 75.5 mm

Commit message: updated firmware
Parts:
- moved J10 122.8 mm to (7.02, 12.0)
- moved J11 122.8 mm to (12.9, 20.5)
- moved J11 122.8 mm to (19.1, 70.0)
- moved J12 122.8 mm to (12.9, 12.5)
- moved J2 122.8 mm to (38.1, 60.7)
- moved J5 122.8 mm to (28.6, 70.0)
- moved J6 122.8 mm to (38.1, 70.0)
- moved J7 122.8 mm to (12.9, 4.52)
- moved J9 122.8 mm to (5.02, 68.0)
- moved J1 122.8 mm to (38.1, 51.0)
- moved J10 122.8 mm to (19.1, 60.4)
- moved J3 122.8 mm to (28.6, 51.0)
- moved J4 122.8 mm to (28.6, 60.4)
- moved J8 122.8 mm to (15.5, 27.4)
- moved J9 122.8 mm to (19.1, 51.0)
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
Commit message: updated pcb :D
Parts:
- removed the J10 at (19.1, 60.4)
- removed the J10 at (7.02, 12.0)
- removed the J11 at (12.9, 20.5)
- removed the J11 at (19.1, 70.0)
- removed the J9 at (5.02, 68.0)
- removed the J9 at (19.1, 51.0)
- added J10: Conn_01x12, JST:JST 1x12, F.Cu at (14.0, 39.5)
- added J11: Conn_01x03, JST:JST 1x3, F.Cu at (26.5, 68.0)
- added J9: Conn_01x06, JST:JST 1x6, F.Cu at (21.5, 51.5)
- J1, J2, J3, J4, J5, J6: footprint Connector:JWT_A3963_1x02_P3.96mm_Vertical -> JST:JST 1x2
- J12, J7: footprint Connector:FanPinHeader_1x03_P2.54mm_Vertical -> JST:JST 1x3
- J8: footprint Connector:FanPinHeader_1x04_P2.54mm_Vertical -> JST:JST 1x4
- moved J12 62.9 mm to (20.0, 75.0), turned to 90 degrees
- moved J3 28.4 mm to (55.0, 61.5)
- moved J4 26.7 mm to (55.0, 64.5)
- moved J5 26.4 mm to (55.0, 68.5)
- moved U3 21.1 mm to (41.0, 57.1)
- moved J7 17.5 mm to (23.5, 18.5)
- moved J1 13.1 mm to (46.0, 61.5)
- moved J2 8.74 mm to (46.0, 64.5)
- moved J6 8.12 mm to (46.0, 68.0)
- moved J8 6.52 mm to (21.5, 30.0), turned to 90 degrees
Routing:
- net GND: track 232.4 -> 0.00 mm
- net BA: track 55.5 -> 10.4 mm
- net +6.5V: track 91.8 -> 47.0 mm
- net BB: track 50.6 -> 10.6 mm
- net +5V: track 77.7 -> 116.9 mm
- net AA: track 38.9 -> 8.33 mm
- net AB: track 34.0 -> 8.33 mm
- net Net-(J10-Pin_2): track 19.3 -> 0.00 mm
- net Net-(J10-Pin_1): track 19.3 -> 0.00 mm
- net Net-(J1-Pin_2): track 19.0 -> 6.50 mm
- net Net-(J1-Pin_1): track 19.0 -> 6.50 mm
- net Net-(J3-Pin_2): track 19.0 -> 7.00 mm
- net Net-(J3-Pin_1): track 19.0 -> 7.00 mm
- net LED1: track 11.0 -> 15.6 mm
- net LED2: track 9.91 -> 12.5 mm
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- removed copper zone on B.Cu, net GND
Other:
- board size 45.5 x 75.5 mm -> 50 x 70 mm

Commit message: updated gbr
Parts:
- moved J9 0.50 mm to (21.5, 52.0)
Routing:
- net +5V: track 116.9 -> 113.0 mm
- net IN2: track 7.71 -> 7.00 mm
- net BA: track 10.4 -> 9.90 mm
Changed lines of the file:
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@@
 		(fp_arc
 			(start 33.249783 -1.367705)
-			(mid 33.285138 -1.35306)
+			(mid 33.285151 -1.353067)
 			(end 33.299783 -1.317705)
 			(stroke
@@
 		(fp_arc
 			(start 23.299783 -1.317705)
-			(mid 23.314428 -1.35306)
+			(mid 23.314428 -1.353063)
 			(end 23.349783 -1.367705)
 			(stroke
@@
 		(fp_arc
 			(start 24.324148 0.462527)
-			(mid 26.469605 -0.023594)
+			(mid 26.469639 -0.023582)
 			(end 24.336385 0.51369)
 			(stroke
@@
 		(fp_arc
 			(start 33.299783 3.582294)
-			(mid 33.285138 3.617649)
+			(mid 33.285139 3.617647)
 			(end 33.249783 3.632294)
 			(stroke
@@
 		(fp_arc
 			(start 23.349783 3.632294)
-			(mid 23.314428 3.617649)
+			(mid 23.314441 3.617643)
 			(end 23.299783 3.582294)
 			(stroke
@@
 		(fp_arc
 			(start 31.667397 6.085796)
-			(mid 32.728057 6.525136)
+			(mid 32.728061 6.525135)
 			(end 33.167397 7.585796)
 			(stroke
@@
 		(fp_arc
 			(start 29.787183 7.399531)
-			(mid 29.726949 7.443544)
+			(mid 29.726945 7.443551)
 			(end 29.653011 7.433617)
 			(stroke
@@
 		(fp_arc
 			(start 29.787183 7.399531)
-			(mid 32.120699 7.132496)
+			(mid 32.120655 7.132547)
 			(end 31.853662 9.466011)
 			(stroke
@@
 		(fp_arc
 			(start 23.981784 7.433617)
-			(mid 26.817397 6.685796)
+			(mid 26.817398 6.685796)
 			(end 29.653011 7.433617)
 			(stroke
@@
 		(fp_arc
 			(start 23.981783 7.433617)
-			(mid 23.907845 7.443544)
+			(mid 23.907859 7.44352)
 			(end 23.847611 7.399531)
 			(stroke
@@
 		(fp_arc
 			(start 20.467397 7.585796)
-			(mid 20.906737 6.525136)
+			(mid 20.906738 6.525137)
 			(end 21.967397 6.085796)
 			(stroke
@@
 		(fp_arc
 			(start 21.781131 9.46601)
-			(mid 21.825145 9.526245)
+			(mid 21.825155 9.526249)
 			(end 21.815218 9.600183)
 			(stroke
@@
 		(fp_arc
 			(start 21.781132 9.466011)
-			(mid 21.514096 7.132496)
+			(mid 21.514101 7.132501)
 			(end 23.847611 7.399531)
 			(stroke
@@
 		(fp_arc
 			(start 31.819576 9.600183)
-			(mid 32.567397 12.435796)
+			(mid 32.567399 12.435797)
 			(end 31.819576 15.27141)
 			(stroke
@@
 		(fp_arc
 			(start 31.819577 9.600184)
-			(mid 31.809649 9.526246)
+			(mid 31.809674 9.526259)
 			(end 31.853662 9.466011)
 			(stroke
@@
 		(fp_arc
 			(start 21.815217 15.271409)
-			(mid 21.825145 15.345347)
+			(mid 21.825126 15.345337)
 			(end 21.781132 15.405582)
 			(stroke
@@
 		(fp_arc
 			(start 21.815218 15.27141)
-			(mid 21.067397 12.435796)
+			(mid 21.067399 12.435797)
 			(end 21.815218 9.600183)
 			(stroke
@@
 		(fp_arc
 			(start 31.853662 15.405582)
-			(mid 32.120698 17.739097)
+			(mid 32.120701 17.739101)
 			(end 29.787183 17.472062)
 			(stroke
@@
 		(fp_arc
 			(start 31.853663 15.405583)
-			(mid 31.809649 15.345348)
+			(mid 31.809646 15.345344)
 			(end 31.819576 15.27141)
 			(stroke
@@
 		(fp_arc
 			(start 13.181636 16.183217)
-			(mid 13.252347 16.212506)
+			(mid 13.252317 16.21252)
 			(end 13.281636 16.283217)
 			(stroke
@@
 		(fp_arc
 			(start 9.481636 16.283217)
-			(mid 9.510925 16.212506)
+			(mid 9.510921 16.212508)
 			(end 9.581636 16.183217)
 			(stroke
@@
 		(fp_arc
 			(start 33.167397 17.285796)
-			(mid 32.728057 18.346456)
+			(mid 32.728058 18.346458)
 			(end 31.667397 18.785796)
 			(stroke
@@
 		(fp_arc
 			(start 29.653011 17.437976)
-			(mid 29.726949 17.428049)
+			(mid 29.726938 17.428069)
 			(end 29.787183 17.472062)
 			(stroke
@@
 		(fp_arc
 			(start 23.847611 17.472062)
-			(mid 21.514095 17.739097)
+			(mid 21.514153 17.739048)
 			(end 21.781132 15.405582)
 			(stroke
@@
 		(fp_arc
 			(start 23.847611 17.472062)
-			(mid 23.907845 17.428049)
+			(mid 23.90785 17.428041)
 			(end 23.981783 17.437976)
 			(stroke
@@
 		(fp_arc
 			(start 13.281636 18.583217)
-			(mid 13.252347 18.653928)
+			(mid 13.252343 18.653929)
 			(end 13.181636 18.683217)
 			(stroke
@@
 		(fp_arc
 			(start 9.581636 18.683217)
-			(mid 9.510925 18.653928)
+			(mid 9.510896 18.653941)
 			(end 9.481636 18.583217)
 			(stroke
@@
 		(fp_arc
 			(start 21.967397 18.785796)
-			(mid 20.906737 18.346456)
+			(mid 20.90674 18.346455)
 			(end 20.467397 17.285796)
 			(stroke
@@
 	(footprint "JST:JST 1x6"
 		(layer "F.Cu")
-		(at 21.5 51.5 90)
+		(at 21.5 52 90)
 		(property "Reference" "J9"
 			(at 0 -0.5 90)
@@
 		(start 43.5 61.5)
 		(end 43.5 68)
-		(width 0.3)
+		(width 0.5)
 		(layer "F.Cu")
 		(net 1)
@@
 		(start 48 61.5)
 		(end 48 68)
-		(width 0.3)
+		(width 0.5)
 		(layer "F.Cu")
 		(net 2)
@@
 		(start 57 61.5)
 		(end 57 68.5)
-		(width 0.3)
+		(width 0.5)
 		(layer "F.Cu")
 		(net 3)
@@
 		(start 52.5 61.5)
 		(end 52.5 68.5)
-		(width 0.3)
+		(width 0.5)
 		(layer "F.Cu")
 		(net 4)
@@
 		(start 28 42.5)
 		(end 21.5 49)
-		(width 0.3)
+		(width 0.5)
 		(layer "F.Cu")
 		(net 5)
@@
 		(start 28 18.5)
 		(end 30 16.5)
-		(width 0.3)
+		(width 0.5)
 		(layer "F.Cu")
 		(net 5)
@@
 		(start 30 16.5)
 		(end 41 16.5)
-		(width 0.3)
+		(width 0.5)
 		(layer "F.Cu")
 		(net 5)
@@
 		(start 28 18.5)
 		(end 28 42.5)
-		(width 0.3)
+		(width 0.5)
 		(layer "F.Cu")
 		(net 5)
-	)
-	(segment
-		(start 26.5 63.5)
-		(end 26.5 63)
-		(width 0.3)
-		(layer "F.Cu")
-		(net 6)
 	)
 	(segment
 		(start 26.5 63.5)
 		(end 48 42)
-		(width 0.3)
+		(width 0.5)
 		(layer "F.Cu")
 		(net 6)
@@
 		(start 14 18.5)
 		(end 19 18.5)
-		(width 0.3)
+		(width 0.5)
 		(layer "F.Cu")
 		(net 6)
@@
 		(start 47 13.5)
 		(end 24 13.5)
-		(width 0.3)
-		(layer "F.Cu")
-		(net 6)
-	)
-	(segment
-		(start 26.5 63.5)
-		(end 32 69)
-		(width 0.3)
+		(width 0.5)
 		(layer "F.Cu")
 		(net 6)
@@
 		(start 24 13.5)
 		(end 19 18.5)
-		(width 0.3)
-		(layer "F.Cu")
-		(net 6)
-	)
-	(segment
-		(start 32 69)
-		(end 32 70.5)
-		(width 0.3)
-		(layer "F.Cu")
-		(net 6)
-	)
-	(segment
-		(start 26.5 63)
-		(end 26 62.5)
-		(width 0.3)
+		(width 0.5)
 		(layer "F.Cu")
 		(net 6)
@@
 		(start 48 42)
 		(end 48 14.5)
-		(width 0.3)
+		(width 0.5)
 		(layer "F.Cu")
 		(net 6)
 	)
 	(segment
-		(start 32 70.5)
+		(start 30.5 67.5)
+		(end 30.5 69.5)
+		(width 0.5)
+		(layer "F.Cu")
+		(net 6)
+	)
+	(segment
+		(start 30.5 69.5)
+		(end 29.5 70.5)
+		(width 0.5)
+		(layer "F.Cu")
+		(net 6)
+	)
+	(segment
+		(start 29.5 70.5)
 		(end 20 70.5)
-		(width 0.3)
+		(width 0.5)
+		(layer "F.Cu")
+		(net 6)
+	)
+	(segment
+		(start 26.5 63.5)
+		(end 30.5 67.5)
+		(width 0.5)
 		(layer "F.Cu")
 		(net 6)
@@
 		(start 48 14.5)
 		(end 47 13.5)
-		(width 0.3)
+		(width 0.5)
 		(layer "F.Cu")
 		(net 6)
@@
 		(start 14 37)
 		(end 21.5 37)
-		(width 0.3)
+		(width 0.5)
 		(layer "F.Cu")
 		(net 8)
@@
 		(start 14 28)
 		(end 21 28)
-		(width 0.3)
-		(layer "F.Cu")
-		(net 9)
-	)
-	(segment
-		(start 21 28)
-		(end 21.5 27.5)
-		(width 0.3)
+		(width 0.5)
 		(layer "F.Cu")
 		(net 9)
@@
 		(start 14 23)
 		(end 21.5 23)
-		(width 0.3)
+		(width 0.5)
 		(layer "F.Cu")
 		(net 10)
@@
 		(start 14 32.5)
 		(end 21.5 32.5)
-		(width 0.3)
+		(width 0.5)
 		(layer "F.Cu")
 		(net 11)
@@
 		(start 14 51)
 		(end 21.5 58.5)
-		(width 0.3)
+		(width 0.5)
 		(layer "F.Cu")
 		(net 12)
@@
 		(start 21.5 44.5)
 		(end 19.5 46.5)
-		(width 0.3)
+		(width 0.5)
 		(layer "F.Cu")
 		(net 13)
@@
 		(start 19.5 46.5)
 		(end 14 46.5)
-		(width 0.3)
+		(width 0.5)
 		(layer "F.Cu")
 		(net 13)
@@
 		(start 16 40)
 		(end 21.5 40)
-		(width 0.3)
+		(width 0.5)
 		(layer "F.Cu")
 		(net 14)
@@
 		(start 14 42)
 		(end 16 40)
-		(width 0.3)
+		(width 0.5)
 		(layer "F.Cu")
 		(net 14)
@@
 		(start 14 56)
 		(end 21 63)
-		(width 0.3)
-		(layer "F.Cu")
-		(net 15)
-	)
-	(segment
-		(start 21 63)
-		(end 21.5 63)
-		(width 0.3)
+		(width 0.5)
 		(layer "F.Cu")
 		(net 15)
@@
 		(start 14 60.5)
 		(end 21.5 68)
-		(width 0.3)
+		(width 0.5)
 		(layer "F.Cu")
 		(net 16)
@@
 		(start 21.5 68)
 		(end 26.5 68)
-		(width 0.3)
+		(width 0.5)
 		(layer "F.Cu")
 		(net 16)
@@
 		(start 14 65)
 		(end 14 69)
-		(width 0.3)
+		(width 0.5)
 		(layer "F.Cu")
 		(net 17)
@@
 		(start 14 69)
 		(end 20 75)
-		(width 0.3)
+		(width 0.5)
 		(layer "F.Cu")
 		(net 17)

Commit message: update gbr pt2
Other:
- board size 50 x 70 mm -> 50 x 71 mm
Changed lines of the file:
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@@
 		(fp_arc
 			(start 23.981783 7.433617)
-			(mid 23.907859 7.44352)
+			(mid 23.907854 7.443509)
 			(end 23.847611 7.399531)
 			(stroke
@@
 		(fp_arc
 			(start 21.781131 9.46601)
-			(mid 21.825155 9.526249)
+			(mid 21.8252 9.526245)
 			(end 21.815218 9.600183)
 			(stroke
@@
 		(fp_arc
 			(start 31.819577 9.600184)
-			(mid 31.809674 9.526259)
+			(mid 31.809685 9.526255)
 			(end 31.853662 9.466011)
 			(stroke
@@
 		(fp_arc
 			(start 13.181636 16.183217)
-			(mid 13.252317 16.21252)
+			(mid 13.252353 16.212514)
 			(end 13.281636 16.283217)
 			(stroke
@@
 		(fp_arc
 			(start 23.847611 17.472062)
-			(mid 23.90785 17.428041)
+			(mid 23.907846 17.427997)
 			(end 23.981783 17.437976)
 			(stroke
@@
 		(fp_arc
 			(start 9.581636 18.683217)
-			(mid 9.510896 18.653941)
+			(mid 9.510931 18.653935)
 			(end 9.481636 18.583217)
 			(stroke
@@
 	)
 	(gr_rect
-		(start 12 12)
+		(start 12 11)
 		(end 62 82)
 		(stroke
